File: PiCard.kicad_pcb (KiCad board)
At the start: 4 copper layers, 101 x 70 mm, 104 parts, among them J1 RS232, J2 Ethernet, J3 Micro_SD_Card_Det2, J4 Bus_M.2_Socket_M, J5 USB_C_Receptacle, J6 USB_C_Receptacle, J8 HDMI_C_1.4, Q2 DMP3013SFV, SW1 SW_DIP_x04, U1 MAX3232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

Commit message: update
Parts:
- moved C23 2.07 mm to (113.0, 82.3)
Connections:
- C23 pad 2: /USB/USB3_VBUS -> +5V
Routing:
- net +5V: track 147.8 -> 149.0 mm, vias 21 -> 22
- net GND: track 247.2 -> 247.9 mm, vias 177 -> 176
- net +3.3V: track 162.5 -> 163.0 mm
Other:
- board size 101 x 70 mm -> 81.5 x 50 mm
