File: Power.kicad_sch (KiCad schematic)
At the start: 36 parts, among them Q2 DMP3013SFV, U6 TPS62180, U7 CYPD3177-24LQ, U8 TPS82130, U9 DS1307Z+, Y1 32.768kHz

Commit message: PiCard v2.2
Parts:
- SYM1: value PiCard v2.1 -> PiCard v2.2
Changed lines of the file:
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@@
 			)
 		)
-		(property "Value" "PiCard v2.1"
+		(property "Value" "PiCard v2.2"
 			(at 206.375 155.575 0)
 			(effects

Commit message: PiCard v3.0
Parts:
- removed BT1: RTC Battery, PiCard:BAT-SMD_MY-1220-03, symbol Device:Battery_Cell
- removed C10, C11: 1u, Capacitor_SMD:C_0603_1608Metric, symbol Device:C
- removed C12, C13: 100n, Capacitor_SMD:C_0402_1005Metric, symbol Device:C
- removed H1, H2: MountingHole, PiCard:MOUNTING-HOLE, symbol Mechanical:MountingHole
- removed JP1: SolderJumper_2_Open, Jumper:SolderJumper-2_P1.3mm_Open_TrianglePad1.0x1.5mm, symbol Jumper:SolderJumper_2_Open
- removed Q2: DMP3013SFV, Package_SON:Diodes_PowerDI3333-8, symbol Transistor_FET:DMP3013SFV
- removed R13, R26, R27: 5.1k, Resistor_SMD:R_0402_1005Metric, symbol Device:R
- removed R25: 1k, Resistor_SMD:R_0402_1005Metric, symbol Device:R
- removed SYM1: PiCard v2.2, PiCard:PICARD_NAMEPLATE, symbol Graphic:Logo_Open_Hardware_Small
- removed U7: CYPD3177-24LQ, Package_DFN_QFN:QFN-24-1EP_4x4mm_P0.5mm_EP2.75x2.75mm, symbol Interface_USB:CYPD3177-24LQ
- removed U9: DS1307Z+, Package_SO:SOIC-8_3.9x4.9mm_P1.27mm, symbol Timer_RTC:DS1307Z+
- removed Y1: 32.768kHz, Crystal:Crystal_SMD_3215-2Pin_3.2x1.5mm, symbol Device:Crystal
- added C17, C21: 100n, Capacitor_SMD:C_0402_1005Metric, symbol Device:C
- added C18: 10u, Capacitor_SMD:C_0805_2012Metric, symbol Device:C
- added C19, C20, C23, C24: 2.2n, Capacitor_SMD:C_0402_1005Metric, symbol Device:C
- added D13, D5, D6: D, Diode_SMD:D_SOD-323, symbol Device:D
- added D3, D8, D9: 1N5819WS, Diode_SMD:D_SOD-323, symbol Device:D_Schottky
- added D4, D7: Zener 20V, Diode_SMD:D_SOD-323, symbol Device:D_Zener
- added R15, R16: 220k 1%, Resistor_SMD:R_0402_1005Metric, symbol Device:R
- added R17, R18: 59k, Resistor_SMD:R_0402_1005Metric, symbol Device:R
- added R19, R20: 28.7k, Resistor_SMD:R_0402_1005Metric, symbol Device:R
- added R21, R22, R24: 953, Resistor_SMD:R_0402_1005Metric, symbol Device:R
- added U10, U9: TVS2200DRV, Package_SON:WSON-6-1EP_2x2mm_P0.65mm_EP1x1.6mm, symbol Power_Protection:TVS2200DRV
- added U11, U12, U16, U17: TPS259470, PiCard:RPW0010A-MFG, symbol PiCard:TPS259470
- added U13, U14, U15, U8: AP21510, Package_DFN_QFN:DFN-6-1EP_2x1.8mm_P0.5mm_EP1.2x1.6mm, symbol PiCard:AP21510FM-7
- C22: value 100n -> 10u; footprint Capacitor_SMD:C_0402_1005Metric -> Capacitor_SMD:C_0805_2012Metric; LCSC C307331 -> C15850; MPN CL05B104KB54PNC -> CL21A106KAYNNNE
- R14: value 1k -> 12k; LCSC C11702 -> C25752; MPN 0402WGF1001TCE -> 0402WGF1202TCE
- R23: value 49.9k -> 953; LCSC C25897 -> C113475; MPN 0402WGF4992TCE -> 0402WGF9530TCE
- renumbered C15 to C10, C16 to C11, C17 to C12, C19 to C13, C20 to C14, C18 to C15, C21 to C16, C14 to C9, R22 to R11, R24 to R12, R15 to R13, U8 to U6, U6 to U7
Connections:
- net +5V: now also C22.1, C17.1, C18.1, C21.1, D4.2 (A), D7.2 (A), U13.2 (IN), U14.2 (IN), U15.2 (IN), U16.5 (IN), U17.5 (IN), U8.2 (IN); no longer C22.2
- net GND: now also C22.2, R23.2, C17.2, C18.2, C19.2, C20.2, C21.2, C23.2, C24.2, D3.2 (A), D8.2 (A), D9.2 (A), R19.2, R20.2, R21.2, R22.2, R24.2, U10.1 (GND), U10.2 (GND), U10.3 (GND), U10.7 (GND), U11.8 (GND), U12.8 (GND), U13.1 (GND), U13.7 (GND), U14.1 (GND), U14.7 (GND), U15.1 (GND), U15.7 (GND), U16.8 (GND), U17.8 (GND), U8.1 (GND), U8.7 (GND), U9.1 (GND), U9.2 (GND), U9.3 (GND), U9.7 (GND); no longer C22.1
- net VBUS: now also D3.1 (K), U11.6 (OUT), U12.6 (OUT); no longer R23.1, U6.1 (EN), U7.E4 (EN)
- net PWR_EN: now reaches R14.1
- net PWR_EN: now also U6.1 (EN), U7.E4 (EN), D13.1 (K)
- new net: D4.1 (K), D5.1 (K)
- new net: C20.1, U12.7 (dVdt)
- new net: R16.2, R18.1, U12.1 (EN/UVLO)
- new net: R18.2, R20.1, U12.2 (OVLO)
- new net: R15.2, R17.1, U11.1 (EN/UVLO)
- new net: R17.2, R19.1, U11.2 (OVLO)
- new net: C19.1, U11.7 (dVdt)
- new net: D6.1 (K), D7.1 (K)
- new net: C24.1, U17.7 (dVdt)
- new net: C23.1, U16.7 (dVdt)
- new net CM_PWR_EN: D13.2 (A)
- new net UCPD1_CC1: U8.5 (OUT), U8.6 (OUT)
- new net UCPD1_CC1_VCONN_EN: U8.3 (EN)
- new net UCPD1_CC2: U13.5 (OUT), U13.6 (OUT)
- new net UCPD1_CC2_VCONN_EN: U13.3 (EN)
- new net UCPD2_CC1: U14.5 (OUT), U14.6 (OUT)
- new net UCPD2_CC1_VCONN_EN: U14.3 (EN)
- new net UCPD2_CC2: U15.5 (OUT), U15.6 (OUT)
- new net UCPD2_CC2_VCONN_EN: U15.3 (EN)
- new net USB0_SINK_ILM: R22.1, U12.9 (ILM)
- new net USB0_SRC_EN: U17.1 (EN/UVLO)
- new net USB0_SRC_ILM: R24.1, U17.9 (ILM)
- new net USB0_SRC_OVLO: U17.2 (OVLO)
- new net USB0_VBUS: D5.2 (A), D8.1 (K), R16.1, U10.4 (IN), U10.5 (IN), U10.6 (IN), U12.5 (IN), U17.6 (OUT)
- new net USB1_SINK_ILM: R21.1, U11.9 (ILM)
- new net USB1_SRC_EN: U16.1 (EN/UVLO)
- new net USB1_SRC_ILM: R23.1, U16.9 (ILM)
- new net USB1_SRC_OVLO: U16.2 (OVLO)
- new net USB1_VBUS: D6.2 (A), D9.1 (K), R15.1, U11.5 (IN), U16.6 (OUT), U9.4 (IN), U9.5 (IN), U9.6 (IN)
- no-connect marks 10 -> 14
Other:
- note removed: "RTC"
- title: (none) -> PiCard
- moved on the sheet: C10, C11, C12, C13, C14, C15, C16, C9, L1, L2, R10, R11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
