File: Power.kicad_sch (KiCad schematic)
At the start: 52 parts, among them U13 TPS259470, U22 TVS2200DRV, U23 TPS259470, U24 TPS259470, U25 TPS259470, U26 TVS2200DRV, U27 AP21510, U28 AP21510, U29 AP21510, U30 AP21510, U6 TPS62180, U8 TPS82130

Commit message: WIP
Parts:
- added D13: D, Diode_SMD:D_SOD-323, symbol Device:D
- C18: renamed from C41; Manufacturer C15850 -> Samsung
- C19: renamed from C38; LCSC (none) -> C1531; MPN (none) -> 0402B222K500NT; Manufacturer (none) -> FH
- C20: renamed from C37; LCSC (none) -> C1531; MPN (none) -> 0402B222K500NT; Manufacturer (none) -> FH
- C22: renamed from C44; Manufacturer C15850 -> Samsung
- C23: renamed from C39; LCSC (none) -> C1531; MPN (none) -> 0402B222K500NT; Manufacturer (none) -> FH
- C24: renamed from C40; LCSC (none) -> C1531; MPN (none) -> 0402B222K500NT; Manufacturer (none) -> FH
- D4: renamed from D12; value D_Zener -> Zener 20V; footprint (none) -> Diode_SMD:D_SOD-323; LCSC (none) -> C19077451; MPN (none) -> BZT52C20S; Manufacturer (none) -> ichjc
- D5: renamed from D11; footprint (none) -> Diode_SMD:D_SOD-323; LCSC (none) -> C2128; MPN (none) -> 1N4148WS; Manufacturer (none) -> CJ
- D6: renamed from D10; footprint (none) -> Diode_SMD:D_SOD-323; LCSC (none) -> C2128; MPN (none) -> 1N4148WS; Manufacturer (none) -> CJ
- D7: renamed from D9; value D_Zener -> Zener 20V; footprint (none) -> Diode_SMD:D_SOD-323; LCSC (none) -> C19077451; MPN (none) -> BZT52C20S; Manufacturer (none) -> ichjc
- R15: renamed from R18; LCSC (none) -> C25767; MPN (none) -> 0402WGF2203TCE; Manufacturer (none) -> Uniroyal
- R16: renamed from R29; LCSC (none) -> C25767; MPN (none) -> 0402WGF2203TCE; Manufacturer (none) -> Uniroyal
- R17: renamed from R19; LCSC (none) -> C32297; MPN (none) -> 0402WGF5902TCE; Manufacturer (none) -> Uniroyal
- R18: renamed from R30; LCSC (none) -> C32297; MPN (none) -> 0402WGF5902TCE; Manufacturer (none) -> Uniroyal
- R19: renamed from R20; LCSC (none) -> C26972; MPN (none) -> 0402WGF2872TCE; Manufacturer (none) -> Uniroyal
- R20: renamed from R31; LCSC (none) -> C26972; MPN (none) -> 0402WGF2872TCE; Manufacturer (none) -> Uniroyal
- R21: renamed from R14; LCSC (none) -> C113475; MPN (none) -> 0402WGF9530TCE; Manufacturer (none) -> Uniroyal
- R22: renamed from R13; LCSC (none) -> C113475; MPN (none) -> 0402WGF9530TCE; Manufacturer (none) -> Uniroyal
- R23: renamed from R16; LCSC (none) -> C113475; MPN (none) -> 0402WGF9530TCE; Manufacturer (none) -> Uniroyal
- R24: renamed from R17; LCSC (none) -> C113475; MPN (none) -> 0402WGF9530TCE; Manufacturer (none) -> Uniroyal
- U10: renamed from U26; LCSC (none) -> C523793; MPN (none) -> TVS2200DRVR; Manufacturer (none) -> Texas Instruments
- U11: renamed from U23; LCSC (none) -> C3662799; MPN (none) -> TPS259470ARPWR; Manufacturer (none) -> Texas Instruments
- U12: renamed from U13; LCSC (none) -> C3662799; MPN (none) -> TPS259470ARPWR; Manufacturer (none) -> Texas Instruments
- U13: renamed from U28; LCSC (none) -> C780752; MPN (none) -> AP21510FM-7; Manufacturer (none) -> DIODES
- U14: renamed from U29; LCSC (none) -> C780752; MPN (none) -> AP21510FM-7; Manufacturer (none) -> DIODES
- U15: renamed from U30; LCSC (none) -> C780752; MPN (none) -> AP21510FM-7; Manufacturer (none) -> DIODES
- U16: renamed from U24; LCSC (none) -> C3662799; MPN (none) -> TPS259470ARPWR; Manufacturer (none) -> Texas Instruments
- U17: renamed from U25; LCSC (none) -> C3662799; MPN (none) -> TPS259470ARPWR; Manufacturer (none) -> Texas Instruments
- U8: renamed from U27; LCSC (none) -> C780752; MPN (none) -> AP21510FM-7; Manufacturer (none) -> DIODES
- U9: renamed from U22; LCSC (none) -> C523793; MPN (none) -> TVS2200DRVR; Manufacturer (none) -> Texas Instruments
- renumbered C15 to C10, C16 to C11, C17 to C12, C19 to C13, C20 to C14, C18 to C15, C21 to C16, C42 to C17, C43 to C21, C14 to C9, D6 to D3, D7 to D9, R22 to R11, R24 to R12, R15 to R13, R32 to R14, U8 to U6, U6 to U7
Connections:
- net PWR_EN: now also D13.1 (K)
- new net CM_PWR_EN: D13.2 (A)
- no-connect marks 6 -> 14
Other:
- title: (none) -> PiCard
- moved on the sheet: R14
