File: module_a.kicad_sch (KiCad schematic)
At the start: 28 parts, among them J1 RS232, J2 Ethernet, J3 Micro_SD_Card_Det2, U1 ADM3101EACPZ, U2 74HC123PW, U3 TPD4EUSB30, U4 TPD4EUSB30, U5 TPS2069C

Commit message: final v3.0
Parts:
- removed U5: TPS2069C, Package_TO_SOT_SMD:SOT-23-5, symbol PiCard:TPS2069C
- added U5: AP2191W, Package_TO_SOT_SMD:SOT-23-5, symbol PiCard:AP2171W
Connections:
- net +3.3V: now also U5.5 (IN)
- net GND: now also U5.2 (GND)
- net SD_PWR: now also U5.1 (OUT)
- net SD_PWR_ON: now also U5.4 (EN)
- net CM_UART4_TX: no longer names the net of ComputeModule1.31 (GPIO12)
- no-connect marks 40 -> 41
Changed lines of the file:
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@@
 	)
 	(junction
-		(at 31.75 175.26)
-		(diameter 0)
-		(color 0 0 0 0)
-	)
-	(junction
 		(at 31.115 86.36)
 		(diameter 0)
@@
 	)
 	(junction
+		(at 31.75 175.26)
+		(diameter 0)
+		(color 0 0 0 0)
+	)
+	(junction
 		(at 33.02 127)
 		(diameter 0)
@@
 	)
 	(no_connect
-		(at 31.75 165.1)
+		(at 52.07 175.26)
 	)
 	(no_connect
@@
 	)
 	(no_connect
+		(at 93.98 60.96)
+	)
+	(no_connect
 		(at 33.02 106.68)
 	)
@@
 	(wire
 		(pts
-			(xy 99.06 60.96) (xy 93.98 60.96)
-		)
-		(stroke
-			(width 0)
-			(type default)
-		)
-	)
-	(wire
-		(pts
 			(xy 154.94 26.67) (xy 149.86 26.67)
 		)
@@
 	(wire
 		(pts
+			(xy 30.48 81.28) (xy 33.02 81.28)
+		)
+		(stroke
+			(width 0)
+			(type default)
+		)
+	)
+	(wire
+		(pts
 			(xy 93.98 30.48) (xy 95.885 30.48)
 		)
@@
 	)
 	(label "SD_PWR"
-		(at 57.15 170.18 0)
+		(at 52.07 170.18 0)
 		(effects
 			(font
@@
 		)
 	)
-	(global_label "CM_UART4_TX"
-		(shape input)
-		(at 99.06 60.96 0)
-		(fields_autoplaced yes)
-		(effects
-			(font
-				(size 1.27 1.27)
-			)
-			(justify left)
-		)
-		(property "Intersheetrefs" "${INTERSHEET_REFS}"
-			(at 114.7451 60.96 0)
-			(effects
-				(font
-					(size 1.27 1.27)
-				)
-				(justify left)
-				(hide yes)
-			)
-		)
-	)
 	(global_label "CM_SPI1_SIO0"
 		(shape input)
@@
 	(global_label "CM_PWR_EN"
 		(shape input)
-		(at 33.02 81.28 180)
+		(at 30.48 81.28 180)
 		(fields_autoplaced yes)
 		(effects
@@
 		)
 		(property "Intersheetrefs" "${INTERSHEET_REFS}"
-			(at 18.9073 81.28 0)
+			(at 16.3673 81.28 0)
 			(effects
 				(font
@@
 	)
 	(symbol
+		(lib_id "PiCard:AP2171W")
+		(at 41.91 172.72 0)
+		(unit 1)
+		(exclude_from_sim no)
+		(in_bom yes)
+		(on_board yes)
+		(dnp no)
+		(fields_autoplaced yes)
+		(property "Reference" "U5"
+			(at 41.91 162.56 0)
+			(effects
+				(font
+					(size 1.27 1.27)
+				)
+			)
+		)
+		(property "Value" "AP2191W"
+			(at 41.91 165.1 0)
+			(effects
+				(font
+					(size 1.27 1.27)
+				)
+			)
+		)
+		(property "Footprint" "Package_TO_SOT_SMD:SOT-23-5"
+			(at 41.91 182.88 0)
+			(effects
+				(font
+					(size 1.27 1.27)
+				)
+				(hide yes)
+			)
+		)
+		(property "Datasheet" "https://www.diodes.com/assets/Datasheets/AP2191.pdf"
+			(at 41.91 171.45 0)
+			(effects
+				(font
+					(size 1.27 1.27)
+				)
+				(hide yes)
+			)
+		)
+		(property "Description" "Current limited power switch, single channel, SOT-23-5"
+			(at 41.91 172.72 0)
+			(effects
+				(font
+					(size 1.27 1.27)
+				)
+				(hide yes)
+			)
+		)
+		(pin "4"
+		)
+		(pin "3"
+		)
+		(pin "1"
+		)
+		(pin "2"
+		)
+		(pin "5"
+		)
+		(instances
+			(project ""
+				(path "/66ede366-7fc2-4b20-87f7-46baaffc82b7/1857bea8-e8dd-4e36-adef-7e084bf0304c"
+					(reference "U5")
+					(unit 1)
+				)
+			)
+		)
+	)
+	(symbol
 		(lib_id "Device:C")
 		(at 149.86 30.48 0)
@@
 	(symbol
 		(lib_id "power:GND")
-		(at 44.45 185.42 0)
+		(at 41.91 180.34 0)
 		(unit 1)
 		(exclude_from_sim no)
@@
 		(dnp no)
 		(property "Reference" "#PWR028"
-			(at 44.45 191.77 0)
+			(at 41.91 186.69 0)
 			(effects
 				(font
@@
 		)
 		(property "Value" "GND"
-			(at 44.577 189.8142 0)
+			(at 42.037 184.7342 0)
 			(effects
 				(font
@@
 		)
 		(property "Footprint" ""
-			(at 44.45 185.42 0)
+			(at 41.91 180.34 0)
 			(effects
 				(font
@@
 		)
 		(property "Datasheet" ""
-			(at 44.45 185.42 0)
+			(at 41.91 180.34 0)
 			(effects
 				(font
@@
 		)
 		(property "Description" ""
-			(at 44.45 185.42 0)
+			(at 41.91 180.34 0)
 			(effects
 				(font
@@
 	(symbol
 		(lib_id "power:+3.3V")
-		(at 57.15 165.1 0)
+		(at 31.75 170.18 90)
 		(unit 1)
 		(exclude_from_sim no)
@@
 		(dnp no)
 		(property "Reference" "#PWR025"
-			(at 57.15 168.91 0)
+			(at 35.56 170.18 0)
 			(effects
 				(font
@@
 		)
 		(property "Value" "+3.3V"
-			(at 60.198 160.528 0)
+			(at 22.86 170.18 90)
 			(effects
 				(font
@@
 		)
 		(property "Footprint" ""
-			(at 57.15 165.1 0)
+			(at 31.75 170.18 0)
 			(effects
 				(font
@@
 		)
 		(property "Datasheet" ""
-			(at 57.15 165.1 0)
+			(at 31.75 170.18 0)
 			(effects
 				(font
@@
 		)
 		(property "Description" ""
-			(at 57.15 165.1 0)
+			(at 31.75 170.18 0)
 			(effects
 				(font
@@
 					(unit 1)
 				)
-			)
-		)
-	)
-	(symbol
-		(lib_id "PiCard:TPS2069C")
-		(at 44.45 170.18 0)
-		(unit 1)
-		(exclude_from_sim no)
-		(in_bom yes)
-		(on_board yes)
-		(dnp no)
-		(fields_autoplaced yes)
-		(property "Reference" "U5"
-			(at 44.45 157.48 0)
-			(effects
-				(font
-					(size 1.27 1.27)
-				)
-			)
-		)
-		(property "Value" "TPS2069C"
-			(at 44.45 160.02 0)
-			(effects
-				(font
-					(size 1.27 1.27)
-				)
-			)
-		)
-		(property "Footprint" "Package_TO_SOT_SMD:SOT-23-5"
-			(at 44.45 157.48 0)
-			(effects
-				(font
-					(size 1.27 1.27)
-				)
-				(hide yes)
-			)
-		)
-		(property "Datasheet" "https://www.ti.com/lit/ds/symlink/tps2069c.pdf"
-			(at 43.18 162.56 0)
-			(effects
-				(font
-					(size 1.27 1.27)
-				)
-				(hide yes)
-			)
-		)
-		(property "Description" "Single power-distribution switcher"
-			(at 44.45 170.18 0)
-			(effects
-				(font
-					(size 1.27 1.27)
-				)
-				(hide yes)
-			)
-		)
-		(property "LCSC" "C181752"
-			(at 44.45 170.18 0)
-			(effects
-				(font
-					(size 1.27 1.27)
-				)
-				(hide yes)
-			)
-		)
-		(property "MPN" "TPS2069CDBVR"
-			(at 44.45 170.18 0)
-			(effects
-				(font
-					(size 1.27 1.27)
-				)
-				(hide yes)
-			)
-		)
-		(property "Manufacturer" "Texas Instruments"
-			(at 44.45 170.18 0)
-			(effects
-				(font
-					(size 1.27 1.27)
-				)
-				(hide yes)
-			)
-		)
-		(pin "3"
-		)
-		(pin "1"
-		)
-		(pin "4"
-		)
-		(pin "5"
-		)
-		(pin "2"
-		)
-		(instances
-			(project ""
-				(path "/66ede366-7fc2-4b20-87f7-46baaffc82b7/1857bea8-e8dd-4e36-adef-7e084bf0304c"
-					(reference "U5")
-					(unit 1)
-				)
