File: USB.kicad_sch (KiCad schematic)
At the start: 29 parts, among them J5 USB_C_Receptacle, J6 USB_C_Receptacle, SW1 SW_DIP_x04, U10 TPS2069C, U11 TPD4EUSB30, U12 TPD4EUSB30, U13 TPD4EUSB30, U14 TPD4EUSB30, U15 TS3USB221, U16 HD3SS3220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

Commit message: Update
Parts:
- removed U10: TPS2069C, Package_TO_SOT_SMD:SOT-23-5, symbol PiCard:TPS2069C
- added C33: 100n, Capacitor_SMD:C_0402_1005Metric, symbol Device:C
- added R16: 15.8k, Resistor_SMD:R_0402_1005Metric, symbol Device:R
- added U10: ~, Package_TO_SOT_SMD:SOT-23-6, symbol PiCard:TPS2553
- U15, U17: footprint PiCard:RSE10 -> Package_DFN_QFN:Texas_UQFN-10_1.5x2mm_P0.5mm
Connections:
- net +5V: now also C33.2, U10.1 (IN); no longer C23.2
- net GND: now also C33.1, R16.2, U10.2 (GND)
- net USB3_VBUS: now also C23.2, U10.6 (OUT)
- net at R28.2: now also U10.3 (EN)
- net VBUS renamed PD_VBUS
- new net: R16.1, U10.5 (ILM)
Other:
- moved on the sheet: C23, C24, C25, C26, C27, C28, C29, C30, C31, C32, J5, J6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

Commit message: update
Connections:
- net +5V: now also C23.2
- net USB3_VBUS: no longer C23.2
Other:
- moved on the sheet: C33, R16, R28, U10
