File: module_b.kicad_sch (KiCad schematic)
At the start: 27 parts, among them J1 Usb Data Jumper, J2 USB_C_Receptacle_USB2.0_16P, M2_3V3 TestPoint, U1 TPD4EUSB30, U7 TPS82130

Commit message: Clean up schematics
Parts:
- C1: Field4 Mouser -> (none); Field5 667-EEF-CX0J101R -> (none); Part Description Capacitor, SP-Cap, 100u, 6.3V, 15mR ESR -> (none)
- C10: Int @ 10 0.206 -> (none); MPN C0402C431J5GACTU -> (none); Mfr KEMET -> (none); SKU 80-C0402C431J5GACTU -> (none); Vendor Mouser -> (none)
- C11, C9: value 0.1uF -> 100nF
- C2, C3, C4, C5, C6, C7: Field4 Digikey -> (none); Field5 490-14381-1-ND -> (none); Field6 GRM21BR71A106KA73L -> (none); Field7 Murata -> (none); Field8 111893011 -> (none); Part Description 10uF 10% 10V Ceramic Capacitor X7R 0805 (2012 Metric) -> (none)
- renumbered PCIe1 to J4
Changed lines of the file:
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@@
       (effects (font (size 1.27 1.27)) hide)
     )
-    (property "Datasheet" "https://search.murata.co.jp/Ceramy/image/img/A01X/G101/ENG/GRM21BR71A106KA73-01.pdf" (at 121.285 172.72 0)
-      (effects (font (size 1.27 1.27)) hide)
-    )
-    (property "Field5" "490-14381-1-ND" (at 121.285 172.72 0)
-      (effects (font (size 1.27 1.27)) hide)
-    )
-    (property "Field4" "Digikey" (at 121.285 172.72 0)
-      (effects (font (size 1.27 1.27)) hide)
-    )
-    (property "Field6" "GRM21BR71A106KA73L" (at 121.285 172.72 0)
-      (effects (font (size 1.27 1.27)) hide)
-    )
-    (property "Field7" "Murata" (at 121.285 172.72 0)
-      (effects (font (size 1.27 1.27)) hide)
-    )
-    (property "Part Description" "	10uF 10% 10V Ceramic Capacitor X7R 0805 (2012 Metric)" (at 121.285 172.72 0)
-      (effects (font (size 1.27 1.27)) hide)
-    )
-    (property "Field8" "111893011" (at 121.285 172.72 0)
+    (property "Datasheet" "" (at 121.285 172.72 0)
       (effects (font (size 1.27 1.27)) hide)
     )
@@
       (effects (font (size 1.27 1.27)) hide)
     )
-    (property "Datasheet" "https://search.murata.co.jp/Ceramy/image/img/A01X/G101/ENG/GRM21BR71A106KA73-01.pdf" (at 255.905 147.955 0)
-      (effects (font (size 1.27 1.27)) hide)
-    )
-    (property "Field5" "490-14381-1-ND" (at 255.905 147.955 0)
-      (effects (font (size 1.27 1.27)) hide)
-    )
-    (property "Field4" "Digikey" (at 255.905 147.955 0)
-      (effects (font (size 1.27 1.27)) hide)
-    )
-    (property "Field6" "GRM21BR71A106KA73L" (at 255.905 147.955 0)
-      (effects (font (size 1.27 1.27)) hide)
-    )
-    (property "Field7" "Murata" (at 255.905 147.955 0)
-      (effects (font (size 1.27 1.27)) hide)
-    )
-    (property "Part Description" "	10uF 10% 10V Ceramic Capacitor X7R 0805 (2012 Metric)" (at 255.905 147.955 0)
-      (effects (font (size 1.27 1.27)) hide)
-    )
-    (property "Field8" "111893011" (at 255.905 147.955 0)
+    (property "Datasheet" "" (at 255.905 147.955 0)
       (effects (font (size 1.27 1.27)) hide)
     )
@@
   (symbol (lib_id "Connector:Bus_M.2_Socket_M") (at 47.625 76.2 0) (mirror y) (unit 1)
     (in_bom yes) (on_board yes) (dnp no)
-    (property "Reference" "PCIe1" (at 45.4309 26.035 0)
+    (property "Reference" "J4" (at 45.4309 26.035 0)
       (effects (font (size 1.27 1.27)) (justify left))
     )
@@
       (project "PiCard"
         (path "/66ede366-7fc2-4b20-87f7-46baaffc82b7/60c6b1bc-0687-463f-9501-11affb2319e2"
-          (reference "PCIe1") (unit 1)
+          (reference "J4") (unit 1)
         )
       )
@@
       (effects (font (size 1.27 1.27)) hide)
     )
-    (property "Int @ 10" "0.206" (at 36.195 170.18 0)
-      (effects (font (size 1.27 1.27)) hide)
-    )
-    (property "MPN" "C0402C431J5GACTU" (at 36.195 170.18 0)
-      (effects (font (size 1.27 1.27)) hide)
-    )
-    (property "Mfr" "KEMET" (at 36.195 170.18 0)
-      (effects (font (size 1.27 1.27)) hide)
-    )
-    (property "SKU" "80-C0402C431J5GACTU" (at 36.195 170.18 0)
-      (effects (font (size 1.27 1.27)) hide)
-    )
-    (property "Vendor" "Mouser" (at 36.195 170.18 0)
-      (effects (font (size 1.27 1.27)) hide)
-    )
     (property "LCSC" "C3875192" (at 36.195 170.18 0)
       (effects (font (size 1.27 1.27)) hide)
@@
       (effects (font (size 1.27 1.27)) (justify left))
     )
-    (property "Value" "0.1uF" (at 143.51 173.99 0)
+    (property "Value" "100nF" (at 143.51 173.99 0)
       (effects (font (size 1.27 1.27)) (justify left))
     )
@@
       (effects (font (size 1.27 1.27)) hide)
     )
-    (property "Datasheet" "https://search.murata.co.jp/Ceramy/image/img/A01X/G101/ENG/GRM21BR71A106KA73-01.pdf" (at 235.585 147.955 0)
-      (effects (font (size 1.27 1.27)) hide)
-    )
-    (property "Field5" "490-14381-1-ND" (at 235.585 147.955 0)
-      (effects (font (size 1.27 1.27)) hide)
-    )
-    (property "Field4" "Digikey" (at 235.585 147.955 0)
-      (effects (font (size 1.27 1.27)) hide)
-    )
-    (property "Field6" "GRM21BR71A106KA73L" (at 235.585 147.955 0)
-      (effects (font (size 1.27 1.27)) hide)
-    )
-    (property "Field7" "Murata" (at 235.585 147.955 0)
-      (effects (font (size 1.27 1.27)) hide)
-    )
-    (property "Part Description" "	10uF 10% 10V Ceramic Capacitor X7R 0805 (2012 Metric)" (at 235.585 147.955 0)
-      (effects (font (size 1.27 1.27)) hide)
-    )
-    (property "Field8" "111893011" (at 235.585 147.955 0)
+    (property "Datasheet" "" (at 235.585 147.955 0)
       (effects (font (size 1.27 1.27)) hide)
     )
@@
       (effects (font (size 1.27 1.27)) hide)
     )
-    (property "Datasheet" "https://search.murata.co.jp/Ceramy/image/img/A01X/G101/ENG/GRM21BR71A106KA73-01.pdf" (at 226.695 147.955 0)
-      (effects (font (size 1.27 1.27)) hide)
-    )
-    (property "Field5" "490-14381-1-ND" (at 226.695 147.955 0)
-      (effects (font (size 1.27 1.27)) hide)
-    )
-    (property "Field4" "Digikey" (at 226.695 147.955 0)
-      (effects (font (size 1.27 1.27)) hide)
-    )
-    (property "Field6" "GRM21BR71A106KA73L" (at 226.695 147.955 0)
-      (effects (font (size 1.27 1.27)) hide)
-    )
-    (property "Field7" "Murata" (at 226.695 147.955 0)
-      (effects (font (size 1.27 1.27)) hide)
-    )
-    (property "Part Description" "	10uF 10% 10V Ceramic Capacitor X7R 0805 (2012 Metric)" (at 226.695 147.955 0)
-      (effects (font (size 1.27 1.27)) hide)
-    )
-    (property "Field8" "111893011" (at 226.695 147.955 0)
+    (property "Datasheet" "" (at 226.695 147.955 0)
       (effects (font (size 1.27 1.27)) hide)
     )
@@
       (effects (font (size 1.27 1.27)) hide)
     )
-    (property "Datasheet" "https://search.murata.co.jp/Ceramy/image/img/A01X/G101/ENG/GRM21BR71A106KA73-01.pdf" (at 130.81 172.72 0)
-      (effects (font (size 1.27 1.27)) hide)
-    )
-    (property "Field5" "490-14381-1-ND" (at 130.81 172.72 0)
-      (effects (font (size 1.27 1.27)) hide)
-    )
-    (property "Field4" "Digikey" (at 130.81 172.72 0)
-      (effects (font (size 1.27 1.27)) hide)
-    )
-    (property "Field6" "GRM21BR71A106KA73L" (at 130.81 172.72 0)
-      (effects (font (size 1.27 1.27)) hide)
-    )
-    (property "Field7" "Murata" (at 130.81 172.72 0)
-      (effects (font (size 1.27 1.27)) hide)
-    )
-    (property "Part Description" "	10uF 10% 10V Ceramic Capacitor X7R 0805 (2012 Metric)" (at 130.81 172.72 0)
-      (effects (font (size 1.27 1.27)) hide)
-    )
-    (property "Field8" "111893011" (at 130.81 172.72 0)
+    (property "Datasheet" "" (at 130.81 172.72 0)
       (effects (font (size 1.27 1.27)) hide)
     )
@@
       (effects (font (size 1.27 1.27)) hide)
     )
-    (property "Datasheet" "https://search.murata.co.jp/Ceramy/image/img/A01X/G101/ENG/GRM21BR71A106KA73-01.pdf" (at 245.745 147.955 0)
-      (effects (font (size 1.27 1.27)) hide)
-    )
-    (property "Field5" "490-14381-1-ND" (at 245.745 147.955 0)
-      (effects (font (size 1.27 1.27)) hide)
-    )
-    (property "Field4" "Digikey" (at 245.745 147.955 0)
-      (effects (font (size 1.27 1.27)) hide)
-    )
-    (property "Field6" "GRM21BR71A106KA73L" (at 245.745 147.955 0)
-      (effects (font (size 1.27 1.27)) hide)
-    )
-    (property "Field7" "Murata" (at 245.745 147.955 0)
-      (effects (font (size 1.27 1.27)) hide)
-    )
-    (property "Part Description" "	10uF 10% 10V Ceramic Capacitor X7R 0805 (2012 Metric)" (at 245.745 147.955 0)
-      (effects (font (size 1.27 1.27)) hide)
-    )
-    (property "Field8" "111893011" (at 245.745 147.955 0)
+    (property "Datasheet" "" (at 245.745 147.955 0)
       (effects (font (size 1.27 1.27)) hide)
     )
@@
       (effects (font (size 1.27 1.27)) hide)
     )
-    (property "Datasheet" "~" (at 212.598 147.955 0)
-      (effects (font (size 1.27 1.27)) hide)
-    )
-    (property "Field4" "Mouser" (at 212.598 147.955 0)
-      (effects (font (size 1.27 1.27)) hide)
-    )
-    (property "Field5" "667-EEF-CX0J101R" (at 212.598 147.955 0)
-      (effects (font (size 1.27 1.27)) hide)
-    )
-    (property "Part Description" "Capacitor, SP-Cap, 100u, 6.3V, 15mR ESR" (at 212.598 147.955 0)
+    (property "Datasheet" "" (at 212.598 147.955 0)
       (effects (font (size 1.27 1.27)) hide)
     )
@@
       (effects (font (size 1.27 1.27)) (justify left))
     )
-    (property "Value" "0.1uF" (at 133.985 173.99 0)
-      (effects (font (size 1.27 1.27)) (justify left))
-    )
+    (property "Value" "100nF" (at 133.985 173.99 0)
+      (effects (font (size 1.27 1.27)) (justify left))
+    )

Commit message: PiCard v2
Parts:
- removed C1: 100uF, Capacitor_Tantalum_SMD:CP_EIA-7343-31_Kemet-D, symbol Device:CP
- removed C10: 430pF, Capacitor_SMD:C_0402_1005Metric, symbol Device:C
- removed C11, C9: 100nF, Capacitor_SMD:C_0603_1608Metric, symbol Device:C
- removed C12, C8: 22uF, Capacitor_SMD:C_0805_2012Metric, symbol Device:C
- removed C2, C3, C4, C5, C6, C7: 10u, Capacitor_SMD:C_0805_2012Metric, symbol Device:C
- removed J1: Usb Data Jumper, Connector_PinHeader_2.00mm:PinHeader_2x02_P2.00mm_Vertical, symbol Connector_Generic:Conn_02x02_Odd_Even
- removed J2: USB_C_Receptacle_USB2.0_16P, PiCard:USB-C-SMD_TYPEC-304J-BCP16, symbol PiCard:USB_C_Receptacle_USB2.0_16P_ALT
- removed M2_3V3, TP3, TP4, TP5: TestPoint, TestPoint:TestPoint_Pad_D2.0mm, symbol Connector:TestPoint
- removed R1: 5.1K, Resistor_SMD:R_0603_1608Metric, symbol Device:R
- removed R2: 5.1K, Capacitor_SMD:C_0603_1608Metric, symbol Device:R
- removed R3, R5: 100k, Resistor_SMD:R_0805_2012Metric, symbol Device:R
- removed R4: 309k, Resistor_SMD:R_0805_2012Metric, symbol Device:R
- removed U1: TPD4EUSB30, Package_SON:USON-10_2.5x1.0mm_P0.5mm, symbol Power_Protection:TPD4EUSB30
- removed U7: TPS82130, PiCard:Texas_SIL0008D_MicroSiP-8-1EP_2.8x3mm_P0.65mm_EP1.1x1.9mm_ThermalVias, symbol Regulator_Switching:TPS82130
- added J8: HDMI_C_1.4, PiCard:HDMI-SMD_19P-P0.40-H-F_HDMI-519S, symbol Connector:HDMI_C_1.4
- added R9: 12k, Resistor_SMD:R_0402_1005Metric, symbol Device:R
- J4: MPN (none) -> APCI0146-P001A; Manufacturer (none) -> LOTES
- renumbered ComputeModule4 to ComputeModule1
Connections:
- net +5V: now also J8.18 (+5V)
- net GND: now also J8.1 (D2S), J8.10 (CKS), J8.13 (GND), J8.4 (D1S), J8.7 (D0S), J8.SH
- net HDMI0_CEC: now reaches ComputeModule1.151 (HDMI0_CEC)
- net HDMI0_CEC: now also J8.14 (CEC)
- net HDMI0_HOT_PLUG: now reaches ComputeModule1.153 (HDMI0_HOTPLUG)
- net HDMI0_HOT_PLUG: now also J8.19 (HPD/HEAC-)
- net CM_USB3_RX_N: now reaches ComputeModule1.157 (DSI0_D0_N)
- net CM_USB3_RX_P: now reaches ComputeModule1.159 (DSI0_D0_P)
- net CM_USB3_USB2_P: now reaches ComputeModule1.163 (DSI0_D1_N)
- net CM_USB3_USB2_N: now reaches ComputeModule1.165 (DSI0_D1_P)
- net CM_USB3_TX_N: now reaches ComputeModule1.169 (DSI0_C_N)
- net HDMI0_TX2_P: now reaches ComputeModule1.170 (HDMI0_TX2_P)
- net HDMI0_TX2_P: now also J8.2 (D2+)
- net CM_USB3_TX_P: now reaches ComputeModule1.171 (DSI0_C_P)
- net HDMI0_TX2_N: now reaches ComputeModule1.172 (HDMI0_TX2_N)
- net HDMI0_TX2_N: now also J8.3 (D2-)
- net HDMI0_TX1_P: now reaches ComputeModule1.176 (HDMI0_TX1_P)
- net HDMI0_TX1_P: now also J8.5 (D1+)
- net HDMI0_TX1_N: now reaches ComputeModule1.178 (HDMI0_TX1_N)
- net HDMI0_TX1_N: now also J8.6 (D1-)
- net HDMI0_TX0_P: now reaches ComputeModule1.182 (HDMI0_TX0_P)
- net HDMI0_TX0_P: now also J8.8 (D0+)
- net HDMI0_TX0_N: now reaches ComputeModule1.184 (HDMI0_TX0_N)
- net HDMI0_TX0_N: now also J8.9 (D0-)
- net HDMI0_CLK_P: now reaches ComputeModule1.188 (HDMI0_CLK_P)
- net HDMI0_CLK_P: now also J8.11 (CK+)
- net HDMI0_CLK_N: now reaches ComputeModule1.190 (HDMI0_CLK_N)
- net HDMI0_CLK_N: now also J8.12 (CK-)
- net HDMI0_SDA: now reaches ComputeModule1.199 (HDMI0_SDA)
- net HDMI0_SDA: now also J8.16 (SDA)
- net HDMI0_SCL: now reaches ComputeModule1.200 (HDMI0_SCL)
- net HDMI0_SCL: now also J8.15 (SCL)
- net M2_3V3 renamed M2_3.3V
- net M2_3.3V: now also R9.2
- net M2_LED: no longer names the net of J4.10 (DAS/~{DSS}/~{LED1})
- net PEWAKE: no longer names the net of J4.54 (~{PEWAKE})
- net PEWAKE: now also R9.1
- net USB2_N renamed CM_USB2_N
- net USB2_P renamed CM_USB2_P
- net USB_OTG_ID: no longer names the net of ComputeModule1.101 (USB_OTG_ID)
- no-connect marks 80 -> 59
Other:
- moved on the sheet: ComputeModule1B

Commit message: wip3
Parts:
- removed J8: HDMI_C_1.4, PiCard:HDMI-SMD_19P-P0.40-H-F_HDMI-519S, symbol Connector:HDMI_C_1.4
- added R38: 3.3k, Resistor_SMD:R_0402_1005Metric, symbol Device:R
Connections:
- net M2_3.3V: now also R38.2
- net M2_LED: now reaches J4.10 (DAS/~{DSS}/~{LED1})
- net M2_SUSCLK: now reaches J4.68 (SUSCLK)
- net M2_SUSCLK: now also R38.1
- net HDMI0_CLK_N: no longer names the net of ComputeModule1.190 (HDMI0_CLK_N)
- net HDMI0_CLK_P: no longer names the net of ComputeModule1.188 (HDMI0_CLK_P)
- net HDMI0_TX0_N: no longer names the net of ComputeModule1.184 (HDMI0_TX0_N)
- net HDMI0_TX0_P: no longer names the net of ComputeModule1.182 (HDMI0_TX0_P)
- net HDMI0_TX1_N: no longer names the net of ComputeModule1.178 (HDMI0_TX1_N)
- net HDMI0_TX1_P: no longer names the net of ComputeModule1.176 (HDMI0_TX1_P)
- net HDMI0_TX2_N: no longer names the net of ComputeModule1.172 (HDMI0_TX2_N)
- net HDMI0_TX2_P: no longer names the net of ComputeModule1.170 (HDMI0_TX2_P)
- no-connect marks 59 -> 56
Other:
- moved on the sheet: J4, R9

Commit message: WIP
Parts:
- ComputeModule1: symbol PiCard:ComputeModule4-CM4 -> PiCard:ComputeModule5-CM5; Field4 Hirose -> Amphenol; Field5 2x DF40C-100DS-0.4V -> 2x 10164227-1001A1RLF
- R9: renamed from R38; LCSC (none) -> C25890; MPN (none) -> 0402WGF3301TCE; Manufacturer (none) -> Uniroyal
- renumbered R9 to R8
Connections:
- net CM_USB_OTG_ID: now reaches ComputeModule1.101 (USB_OTG_ID)
- net CM_USB3_0_SS_RX-: now reaches ComputeModule1.128 (USB3-0-RX_N)
- net CM_USB3_0_SS_RX+: now reaches ComputeModule1.130 (USB3-0-RX_P)
- net CM_USB3_0_HS_D+: now reaches ComputeModule1.134 (USB3-0-D_P)
- net CM_USB3_0_HS_D-: now reaches ComputeModule1.136 (USB3-0-D_N)
- net CM_USB3_0_SS_TX-: now reaches ComputeModule1.140 (USB3-0-TX_N)
- net CM_USB3_0_SS_TX+: now reaches ComputeModule1.142 (USB3-0-TX_P)
- net CM_USB2_N renamed CM_USB2_D-
- net CM_USB2_P renamed CM_USB2_D+
- net CM_USB3_RX_N renamed CM_USB3_1_SS_RX-
- net CM_USB3_RX_P renamed CM_USB3_1_SS_RX+
- net CM_USB3_TX_N renamed CM_USB3_1_SS_TX+
- net CM_USB3_TX_P renamed CM_USB3_1_SS_TX-
- net CM_USB3_USB2_N renamed CM_USB3_1_HS_D-
- net CM_USB3_USB2_P renamed CM_USB3_1_HS_D+
- net HDMI0_CEC: no longer names the net of ComputeModule1.151 (HDMI0_CEC)
- net HDMI0_HOT_PLUG: no longer names the net of ComputeModule1.153 (HDMI0_HOTPLUG)
- net HDMI0_SCL: no longer names the net of ComputeModule1.200 (HDMI0_SCL)
- net HDMI0_SDA: no longer names the net of ComputeModule1.199 (HDMI0_SDA)
- no-connect marks 56 -> 61
Other:
- title: (none) -> PiCard
- moved on the sheet: ComputeModule1B
